Commit message: update robot_name to frame

File: description/lidar.xacro (robot description, xacro)
@@ -2,9 +2,9 @@
 <robot xmlns:xacro="http://www.ros.org/wiki/xacro" >
     <joint name="laser_joint" type="fixed">
-        <parent link="base_link"/>
-        <child link="laser_frame"/>
+        <parent link="${robot_name}/base_link"/>
+        <child link="${robot_name}/laser_frame"/>
         <origin xyz="0.115 0 0.25" rpy="0 0 0"/>
     </joint>
-    <link name="laser_frame">
+    <link name="${robot_name}/laser_frame">
         <visual>
             <geometry>

File: description/robot_core.xacro (robot description, xacro)
@@ -3,4 +3,5 @@
     <xacro:include filename="inertial_macros.xacro"/>
     <xacro:include filename="omniwheel_macros.xacro"/>
+    <xacro:property name="robot_name" value="nunbot"/>
     <!-- Robot dimensions -->
     <xacro:property name="chassis_diameter" value="0.315"/>
@@ -29,22 +30,23 @@
         <color rgba="1 0 0 1"/>
     </material>
-    <!-- BASE LINK -->
-    <link name="base_link">
+    <!-- BASE_FOOTPRINT LINK -->
+    <link name="${robot_name}/base_footprint">
     </link>
     <!-- BASE_FOOTPRINT LINK -->
     <joint name="base_footprint_joint" type="fixed">
-        <parent link="base_link"/>
-        <child link="base_footprint"/>
+        <parent link="${robot_name}/base_footprint"/>
+        <child link="${robot_name}/base_link"/>
         <origin xyz="0 0 0" rpy="0 0 0"/>
     </joint>
-    <link name="base_footprint">
+    <!-- BASE LINK -->
+    <link name="${robot_name}/base_link">
     </link>
     <!-- CHASSIS LINK -->
     <joint name="chassis_joint" type="fixed">
-        <parent link="base_link"/>
-        <child link="chassis"/>
+        <parent link="${robot_name}/base_link"/>
+        <child link="${robot_name}/chassis"/>
         <origin xyz="0 0 ${wheel_radius+0.01}"/>
     </joint>
-    <link name="chassis">
+    <link name="${robot_name}/chassis">
         <visual>
             <origin xyz="0 0 ${chassis_height/2}"/>
@@ -64,10 +66,10 @@
         </xacro:inertial_cylinder>
     </link>
-    <gazebo reference="chassis">
+    <gazebo reference="${robot_name}/chassis">
         <material>Gazebo/Orange</material>
     </gazebo>
     <!-- Wheels-->
-    <xacro:omni_wheel name="wheel_1" parent="base_link" angle_deg="60" yaw="${pi-pi/6}"/>
-    <xacro:omni_wheel name="wheel_2" parent="base_link" angle_deg="180" yaw="${-pi/2}"/>
-    <xacro:omni_wheel name="wheel_3" parent="base_link" angle_deg="300" yaw="${pi/6}"/>
+    <xacro:omni_wheel name="${robot_name}/wheel_1" parent="${robot_name}/base_link" angle_deg="60" yaw="${pi-pi/6}"/>
+    <xacro:omni_wheel name="${robot_name}/wheel_2" parent="${robot_name}/base_link" angle_deg="180" yaw="${-pi/2}"/>
+    <xacro:omni_wheel name="${robot_name}/wheel_3" parent="${robot_name}/base_link" angle_deg="300" yaw="${pi/6}"/>
 </robot>

File: description/sensors.xacro (robot description, xacro)
@@ -2,16 +2,16 @@
 <robot xmlns:xacro="http://www.ros.org/wiki/xacro" >
     <joint name="imu_joint" type="fixed">
-        <parent link="base_link"/>
-        <child link="imu_link"/>
+        <parent link="${robot_name}/base_link"/>
+        <child link="${robot_name}/imu_link"/>
         <origin xyz="0 0 0.15" rpy="0 0 ${-pi / 4}"/>
     </joint>
-    <link name="imu_link">
+    <link name="${robot_name}/imu_link">
     </link>
     <joint name="camera_joint" type="fixed">
-        <parent link="base_link"/>
-        <child link="camera_link"/>
+        <parent link="${robot_name}/base_link"/>
+        <child link="${robot_name}/camera_link"/>
         <origin xyz="0.14 0.05 0.15" rpy="${pi / 2} 0 ${pi / 2}"/>
     </joint>
-    <link name="camera_link">
+    <link name="${robot_name}/camera_link">
     </link>
 </robot>

Commit message: update config files

File: description/lidar.xacro (robot description, xacro)
@@ -4,5 +4,5 @@
         <parent link="${robot_name}/base_link"/>
         <child link="${robot_name}/laser_frame"/>
-        <origin xyz="0.115 0 0.25" rpy="0 0 0"/>
+        <origin xyz="0.115 0 0.25" rpy="0 0 ${pi}"/>
     </joint>
     <link name="${robot_name}/laser_frame">
